File: Board/address.kicad_sch (KiCad schematic)
At the start: 10 parts, among them U1 74LS257, U12 74LS273, U13 74LS273, U2 74LS257, U3 74LS257, U4 74LS257, U5 74LS283, U6 74LS283, U7 74LS283, U8 74LS283

Commit message: more work on the frontpanel
Other:
- note added: "CSA-FRONTPANEL-1.0A"
Changed lines of the file:
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@@
 	(generator_version "10.0")
 	(paper "A3")
+	(text "CSA-FRONTPANEL-1.0A"
+		(exclude_from_sim no)
+		(at 323.215 262.255 0)
+		(effects
+			(font
+				(size 3.81 3.2385)
+			)
+			(justify left bottom)
+		)
+	)
 	(junction
 		(at 193.675 88.9)
