File: Board/Board.kicad_pcb (KiCad board)
At the start: 2 copper layers, 124 parts, among them J2 Conn_02x25_Odd_Even, SW1 SW_SPST, SW10 SW_SPDT, SW11 SW_SPDT, SW12 SW_SPDT, SW13 SW_SPDT, SW14 SW_SPDT, SW15 SW_SPDT, SW16 SW_SPDT, SW17 SW_SPDT, SW18 SW_SPST, SW19 SW_SPST, SW2 SW_SPDT, SW20 SW_SPST, SW3 SW_SPDT, SW4 SW_SPDT, SW5 SW_SPDT, SW6 SW_SPDT, SW7 SW_SPDT, SW8 SW_SPDT, SW9 SW_SPDT, U1 74LS257, U10 74LS257, U11 74LS08, U12 74LS273, U13 74LS273, U14 74LS245, U15 74LS245, U16 74LS245, U17 74LS245, U18 74LS245, U19 74LS14, U2 74LS257, U20 74HCT00, U21 74HCT74, U22 74HCT74, U23 74HCT02, U24 74LS273, U3 74LS257, U4 74LS257, U5 74LS283, U6 74LS283, U7 74LS283, U8 74LS283, U9 74LS257

Commit message: more work on the frontpanel
Parts:
- added D25: LED, LED_SMD:LED_0603_1608Metric_Pad1.05x0.95mm_HandSolder, F.Cu at (178.7, 82.1)
- added D26: LED, LED_SMD:LED_0603_1608Metric_Pad1.05x0.95mm_HandSolder, F.Cu at (178.7, 84.7)
- added D27: LED, LED_SMD:LED_0603_1608Metric_Pad1.05x0.95mm_HandSolder, F.Cu at (178.7, 87.3)
- added D28: LED, LED_SMD:LED_0805_2012Metric_Pad1.15x1.40mm_HandSolder, F.Cu at (230.0, 96.3)
- added D29: LED, LED_SMD:LED_0603_1608Metric_Pad1.05x0.95mm_HandSolder, F.Cu at (213.3, 113.1)
- added D30: LED, LED_SMD:LED_0603_1608Metric_Pad1.05x0.95mm_HandSolder, F.Cu at (213.3, 115.7)
- added D31: LED, LED_SMD:LED_0603_1608Metric_Pad1.05x0.95mm_HandSolder, F.Cu at (213.3, 118.2)
- added D32: LED, LED_SMD:LED_0603_1608Metric_Pad1.05x0.95mm_HandSolder, F.Cu at (213.3, 120.8)
- added D33: LED, LED_SMD:LED_0603_1608Metric_Pad1.05x0.95mm_HandSolder, F.Cu at (213.3, 123.4)
- added D34: LED, LED_SMD:LED_0603_1608Metric_Pad1.05x0.95mm_HandSolder, F.Cu at (213.3, 126.0)
- added D35: LED, LED_SMD:LED_0603_1608Metric_Pad1.05x0.95mm_HandSolder, F.Cu at (217.7, 113.1)
- added D36: LED, LED_SMD:LED_0603_1608Metric_Pad1.05x0.95mm_HandSolder, F.Cu at (217.7, 115.7)
- added D37: LED, LED_SMD:LED_0603_1608Metric_Pad1.05x0.95mm_HandSolder, F.Cu at (217.7, 118.2)
- added D38: LED, LED_SMD:LED_0603_1608Metric_Pad1.05x0.95mm_HandSolder, F.Cu at (217.7, 120.8)
- added D39: LED, LED_SMD:LED_0603_1608Metric_Pad1.05x0.95mm_HandSolder, F.Cu at (217.7, 123.4)
- added D40: LED, LED_SMD:LED_0603_1608Metric_Pad1.05x0.95mm_HandSolder, F.Cu at (217.7, 126.0)
- added D41: LED, LED_SMD:LED_0603_1608Metric_Pad1.05x0.95mm_HandSolder, F.Cu at (222.1, 113.1)
- added D42: LED, LED_SMD:LED_0603_1608Metric_Pad1.05x0.95mm_HandSolder, F.Cu at (222.1, 115.7)
- added D43: LED, LED_SMD:LED_0603_1608Metric_Pad1.05x0.95mm_HandSolder, F.Cu at (222.1, 118.2)
- added D44: LED, LED_SMD:LED_0603_1608Metric_Pad1.05x0.95mm_HandSolder, F.Cu at (222.1, 120.8)
- added J3: Conn_02x08_Odd_Even, Connector_IDC:IDC-Header_2x08_P2.54mm_Vertical, F.Cu at (152.3, 86.9)
- added R49: 10k, Resistor_SMD:R_0603_1608Metric_Pad0.98x0.95mm_HandSolder, F.Cu at (169.9, 99.6)
- added R50: 10k, Resistor_SMD:R_0603_1608Metric_Pad0.98x0.95mm_HandSolder, F.Cu at (174.3, 82.0)
- added R51: 560, Resistor_SMD:R_0603_1608Metric_Pad0.98x0.95mm_HandSolder, F.Cu at (174.3, 84.5)
- added R52: 560, Resistor_SMD:R_0603_1608Metric_Pad0.98x0.95mm_HandSolder, F.Cu at (174.3, 87.1)
- added R53: 560, Resistor_SMD:R_0603_1608Metric_Pad0.98x0.95mm_HandSolder, F.Cu at (229.8, 99.0)
- added R54: 10k, Resistor_SMD:R_0603_1608Metric_Pad0.98x0.95mm_HandSolder, F.Cu at (174.3, 89.6)
- added R55: 560, Resistor_SMD:R_0603_1608Metric_Pad0.98x0.95mm_HandSolder, F.Cu at (174.3, 92.1)
- added R56: 560, Resistor_SMD:R_0603_1608Metric_Pad0.98x0.95mm_HandSolder, F.Cu at (226.4, 113.0)
- added R57: 560, Resistor_SMD:R_0603_1608Metric_Pad0.98x0.95mm_HandSolder, F.Cu at (226.4, 115.5)
- added R58: 560, Resistor_SMD:R_0603_1608Metric_Pad0.98x0.95mm_HandSolder, F.Cu at (226.4, 118.0)
- added R59: 560, Resistor_SMD:R_0603_1608Metric_Pad0.98x0.95mm_HandSolder, F.Cu at (226.4, 120.6)
- added R60: 560, Resistor_SMD:R_0603_1608Metric_Pad0.98x0.95mm_HandSolder, F.Cu at (226.4, 123.1)
- added R61: 560, Resistor_SMD:R_0603_1608Metric_Pad0.98x0.95mm_HandSolder, F.Cu at (226.4, 125.6)
- added R62: 560, Resistor_SMD:R_0603_1608Metric_Pad0.98x0.95mm_HandSolder, F.Cu at (230.8, 113.0)
- added R63: 560, Resistor_SMD:R_0603_1608Metric_Pad0.98x0.95mm_HandSolder, F.Cu at (230.8, 115.5)
- added R64: 560, Resistor_SMD:R_0603_1608Metric_Pad0.98x0.95mm_HandSolder, F.Cu at (230.8, 118.0)
- added R65: 560, Resistor_SMD:R_0603_1608Metric_Pad0.98x0.95mm_HandSolder, F.Cu at (230.8, 120.6)
- added R66: 560, Resistor_SMD:R_0603_1608Metric_Pad0.98x0.95mm_HandSolder, F.Cu at (230.8, 123.1)
- added R67: 560, Resistor_SMD:R_0603_1608Metric_Pad0.98x0.95mm_HandSolder, F.Cu at (230.8, 125.6)
- added R68: 560, Resistor_SMD:R_0603_1608Metric_Pad0.98x0.95mm_HandSolder, F.Cu at (235.1, 113.0)
- added R69: 560, Resistor_SMD:R_0603_1608Metric_Pad0.98x0.95mm_HandSolder, F.Cu at (235.1, 115.5)
- added R70: 560, Resistor_SMD:R_0603_1608Metric_Pad0.98x0.95mm_HandSolder, F.Cu at (235.1, 118.0)
- added R71: 560, Resistor_SMD:R_0603_1608Metric_Pad0.98x0.95mm_HandSolder, F.Cu at (235.1, 120.6)
- added SW21: SW_SPDT, Library:SW_K4625, F.Cu at (180.6, 116.0)
- added U25: 74LS245, Package_SO:TSSOP-20_4.4x5mm_P0.5mm, F.Cu at (229.0, 130.1)
- added U26: 74LS06, Package_SO:SOIC-14_3.9x8.7mm_P1.27mm, F.Cu at (186.1, 106.1)
- added U27: 74LS245, Package_SO:TSSOP-20_4.4x5mm_P0.5mm, F.Cu at (229.0, 136.7)
- D1, D10, D11, D12, D13, D14, D15, D16, D2, D3, D4, D5, D6, D7, D8, D9: footprint LED_SMD:LED_0603_1608Metric_Pad1.05x0.95mm_HandSolder -> LED_SMD:LED_0805_2012Metric_Pad1.15x1.40mm_HandSolder
- R17, R18, R19, R20, R21, R22, R23, R24, R25, R26, R27, R28, R29, R30, R31, R32, R41, R42, R43, R44, R45, R46, R47, R48: value 10k -> 560
- U11: value 74LS08 -> 74LS32; footprint Package_CSP:Xilinx_CSG48_7.0x7.0mm_Layout7x7_P0.8mm -> Package_SO:SOIC-14_3.9x8.7mm_P1.27mm
- U20, U21, U22, U23: footprint Package_CSP:Xilinx_CSG48_7.0x7.0mm_Layout7x7_P0.8mm -> Package_SO:SOIC-14_3.9x8.7mm_P1.27mm
- moved R26 79.3 mm to (165.6, 82.0)
- moved R27 79.3 mm to (165.6, 84.5)
- moved R28 79.3 mm to (165.6, 87.1)
- moved R18 78.9 mm to (161.2, 82.0)
- moved R19 78.9 mm to (161.2, 84.5)
- moved R20 78.9 mm to (161.2, 87.1)
- moved R21 78.9 mm to (161.2, 89.6)
- moved R22 78.9 mm to (161.2, 92.1)
- moved R23 75.2 mm to (161.2, 94.6)
- moved R24 75.2 mm to (161.2, 97.1)
- moved R25 75.2 mm to (161.2, 99.6)
- moved R29 74.7 mm to (165.6, 89.6)
- moved R30 74.7 mm to (165.6, 92.1)
- moved R31 74.7 mm to (165.6, 94.6)
- moved R32 74.7 mm to (165.6, 97.1)
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Connections:
- net Net-(SW1-B) renamed /RESIN
- net Net-(SW20-B) renamed CLKIN
- D1 pad 1: Net-(D1-K) -> D0IN
- D1 pad 2: ID0 -> Net-(D1-A)
- D2 pad 1: Net-(D2-K) -> D1IN
- D2 pad 2: ID1 -> Net-(D2-A)
- D3 pad 1: Net-(D3-K) -> D2IN
- D3 pad 2: ID2 -> Net-(D3-A)
- D4 pad 1: Net-(D4-K) -> D3IN
- D4 pad 2: ID3 -> Net-(D4-A)
- D5 pad 1: Net-(D5-K) -> D4IN
- D5 pad 2: ID4 -> Net-(D5-A)
- D6 pad 1: Net-(D6-K) -> D5IN
- D6 pad 2: ID5 -> Net-(D6-A)
- D7 pad 1: Net-(D7-K) -> D6IN
- D7 pad 2: ID6 -> Net-(D7-A)
- D8 pad 1: Net-(D8-K) -> D7IN
- D8 pad 2: ID7 -> Net-(D8-A)
- J2 pad 10: unconnected-(J2-Pin_10-Pad10) -> /BBE
- J2 pad 11: unconnected-(J2-Pin_11-Pad11) -> BA13
- J2 pad 12: unconnected-(J2-Pin_12-Pad12) -> BA14
- J2 pad 13: unconnected-(J2-Pin_13-Pad13) -> BD7
- J2 pad 14: unconnected-(J2-Pin_14-Pad14) -> BA11
- J2 pad 15: unconnected-(J2-Pin_15-Pad15) -> BA12
- J2 pad 16: unconnected-(J2-Pin_16-Pad16) -> BD6
- J2 pad 17: unconnected-(J2-Pin_17-Pad17) -> BA9
- J2 pad 18: unconnected-(J2-Pin_18-Pad18) -> BA10
- J2 pad 19: unconnected-(J2-Pin_19-Pad19) -> BD5
- J2 pad 20: unconnected-(J2-Pin_20-Pad20) -> BA7
- J2 pad 21: unconnected-(J2-Pin_21-Pad21) -> BA8
- J2 pad 22: unconnected-(J2-Pin_22-Pad22) -> BD4
- J2 pad 23: unconnected-(J2-Pin_23-Pad23) -> BA5
- J2 pad 24: unconnected-(J2-Pin_24-Pad24) -> BA6
- J2 pad 25: unconnected-(J2-Pin_25-Pad25) -> BD3
- J2 pad 26: unconnected-(J2-Pin_26-Pad26) -> BA3
- J2 pad 27: unconnected-(J2-Pin_27-Pad27) -> BA4
- J2 pad 28: unconnected-(J2-Pin_28-Pad28) -> BD2
- J2 pad 29: unconnected-(J2-Pin_29-Pad29) -> BA1
- J2 pad 3: unconnected-(J2-Pin_3-Pad3) -> BA19
- J2 pad 30: unconnected-(J2-Pin_30-Pad30) -> BA2
- J2 pad 31: unconnected-(J2-Pin_31-Pad31) -> BD1
- J2 pad 32: unconnected-(J2-Pin_32-Pad32) -> BSYNC
- J2 pad 33: unconnected-(J2-Pin_33-Pad33) -> BA0
- J2 pad 34: unconnected-(J2-Pin_34-Pad34) -> BD0
- J2 pad 35: unconnected-(J2-Pin_35-Pad35) -> BR/-W
- J2 pad 36: unconnected-(J2-Pin_36-Pad36) -> BPHI2
- J2 pad 37: unconnected-(J2-Pin_37-Pad37) -> /BNMI
- J2 pad 38: unconnected-(J2-Pin_38-Pad38) -> BRDY
- J2 pad 39: unconnected-(J2-Pin_39-Pad39) -> BPHI1
- J2 pad 4: unconnected-(J2-Pin_4-Pad4) -> /BMEMSEL
- J2 pad 40: unconnected-(J2-Pin_40-Pad40) -> /BIRQ
- J2 pad 41: unconnected-(J2-Pin_41-Pad41) -> BV33
- J2 pad 42: unconnected-(J2-Pin_42-Pad42) -> BPHI2
- J2 pad 43: unconnected-(J2-Pin_43-Pad43) -> /BRES
- J2 pad 44: unconnected-(J2-Pin_44-Pad44) -> VBUF
- J2 pad 45: unconnected-(J2-Pin_45-Pad45) -> B2PHI2
- J2 pad 46: unconnected-(J2-Pin_46-Pad46) -> GND
- J2 pad 47: unconnected-(J2-Pin_47-Pad47) -> B8PHI2
- J2 pad 48: unconnected-(J2-Pin_48-Pad48) -> VCC
- J2 pad 49: unconnected-(J2-Pin_49-Pad49) -> GND
- J2 pad 5: unconnected-(J2-Pin_5-Pad5) -> BA17
- J2 pad 50: unconnected-(J2-Pin_50-Pad50) -> VCC
- J2 pad 6: unconnected-(J2-Pin_6-Pad6) -> BA18
- J2 pad 7: unconnected-(J2-Pin_7-Pad7) -> /BIOSEL
- J2 pad 8: unconnected-(J2-Pin_8-Pad8) -> BA15
- J2 pad 9: unconnected-(J2-Pin_9-Pad9) -> BA14
- R1 pad 1: ID0 -> VCC
- R1 pad 2: GND -> D0IN
- R17 pad 1: Net-(D1-K) -> Net-(D1-A)
- R17 pad 2: GND -> VCC
- R18 pad 1: Net-(D2-K) -> Net-(D2-A)
- R18 pad 2: GND -> VCC
- R19 pad 1: Net-(D3-K) -> Net-(D3-A)
- R19 pad 2: GND -> VCC
- R2 pad 1: ID1 -> D1IN
- R2 pad 2: GND -> VCC
- R20 pad 1: Net-(D4-K) -> Net-(D4-A)
- R20 pad 2: GND -> VCC
- R21 pad 1: Net-(D5-K) -> Net-(D5-A)
- R21 pad 2: GND -> VCC
- R22 pad 1: Net-(D6-K) -> Net-(D6-A)
- R22 pad 2: GND -> VCC
- R23 pad 1: Net-(D7-K) -> Net-(D7-A)
- R23 pad 2: GND -> VCC
- R24 pad 1: Net-(D8-K) -> Net-(D8-A)
- R24 pad 2: GND -> VCC
- R3 pad 1: ID2 -> D2IN
- R3 pad 2: GND -> VCC
- R4 pad 1: ID3 -> D3IN
- R4 pad 2: GND -> VCC
- R41 pad 1: Net-(D17-K) -> Net-(D18-K)
- R42 pad 1: Net-(D18-K) -> Net-(D19-K)
- R43 pad 1: Net-(D19-K) -> Net-(D20-K)
- R44 pad 1: Net-(D20-K) -> Net-(D21-K)
- R45 pad 1: Net-(D21-K) -> Net-(D22-K)
- R46 pad 1: Net-(D22-K) -> Net-(D23-K)
- R47 pad 1: Net-(D23-K) -> Net-(D24-K)
- R48 pad 1: Net-(D24-K) -> Net-(R48-Pad1)
- R48 pad 2: GND -> Net-(D27-K)
- R5 pad 1: ID4 -> D4IN
- R5 pad 2: GND -> VCC
- R6 pad 1: ID5 -> D5IN
- R6 pad 2: GND -> VCC
- R7 pad 1: ID6 -> D6IN
- R7 pad 2: GND -> VCC
- R8 pad 1: ID7 -> D7IN
- R8 pad 2: GND -> VCC
- SW2 pad 1: VCC -> unconnected-(SW2-A-Pad1)
- SW2 pad 2: ID0 -> D0IN
- SW2 pad 3: unconnected-(SW2-C-Pad3) -> GND
- SW3 pad 1: VCC -> unconnected-(SW3-A-Pad1)
- SW3 pad 2: ID1 -> D1IN
- SW3 pad 3: unconnected-(SW3-C-Pad3) -> GND
- SW4 pad 1: VCC -> unconnected-(SW4-A-Pad1)
- SW4 pad 2: ID2 -> D2IN
- SW4 pad 3: unconnected-(SW4-C-Pad3) -> GND
- SW5 pad 1: VCC -> unconnected-(SW5-A-Pad1)
- SW5 pad 2: ID3 -> D3IN
- SW5 pad 3: unconnected-(SW5-C-Pad3) -> GND
- SW6 pad 1: VCC -> unconnected-(SW6-A-Pad1)
- SW6 pad 2: ID4 -> D4IN
- SW6 pad 3: unconnected-(SW6-C-Pad3) -> GND
- SW7 pad 1: VCC -> unconnected-(SW7-A-Pad1)
- SW7 pad 2: ID5 -> D5IN
- SW7 pad 3: unconnected-(SW7-C-Pad3) -> GND
- SW8 pad 1: VCC -> unconnected-(SW8-A-Pad1)
- SW8 pad 2: ID6 -> D6IN
- SW8 pad 3: unconnected-(SW8-C-Pad3) -> GND
- SW9 pad 1: VCC -> unconnected-(SW9-A-Pad1)
- SW9 pad 2: ID7 -> D7IN
- SW9 pad 3: unconnected-(SW9-C-Pad3) -> GND
- U1 pad 11: ID3 -> D3IN
- U1 pad 14: ID2 -> D2IN
- U1 pad 2: ID0 -> D0IN
- U1 pad 5: ID1 -> D1IN
- U10 pad 11: ID7 -> D7IN
- U10 pad 14: ID6 -> D6IN
- U10 pad 2: ID4 -> D4IN
- U10 pad 5: ID5 -> D5IN
- U19 pad 10: /RES -> Net-(U21A-C)
- U19 pad 11: RES -> CLKD
- U19 pad 12: (no net) -> Net-(U11-Pad12)
- U19 pad 13: (no net) -> BRDY
- U2 pad 11: ID7 -> D7IN
- U2 pad 14: ID6 -> D6IN
- U2 pad 2: ID4 -> D4IN
- U2 pad 5: ID5 -> D5IN
- U3 pad 11: ID3 -> D3IN
- U3 pad 14: ID2 -> D2IN
- U3 pad 2: ID0 -> D0IN
- U3 pad 5: ID1 -> D1IN
- U4 pad 11: ID7 -> D7IN
- U4 pad 14: ID6 -> D6IN
- U4 pad 2: ID4 -> D4IN
- U4 pad 5: ID5 -> D5IN
- U9 pad 11: ID3 -> D3IN
- U9 pad 14: ID2 -> D2IN
- U9 pad 2: ID0 -> D0IN
- U9 pad 5: ID1 -> D1IN

Commit message: More work
Parts:
- removed C4, C5: 100n, Capacitor_SMD:C_0603_1608Metric_Pad1.08x0.95mm_HandSolder
- removed D28: LED, LED_SMD:LED_0805_2012Metric_Pad1.15x1.40mm_HandSolder
- removed R35, R37: 1k, Resistor_SMD:R_0603_1608Metric_Pad0.98x0.95mm_HandSolder
- removed R36, R38, R50: 10k, Resistor_SMD:R_0603_1608Metric_Pad0.98x0.95mm_HandSolder
- removed R53: 560, Resistor_SMD:R_0603_1608Metric_Pad0.98x0.95mm_HandSolder
- removed SW18, SW19: SW_SPST, Button_Switch_THT:SW_TH_Tactile_Omron_B3F-107x
- removed SW21: SW_SPDT, Library:SW_K4625
- removed U10, U9: 74LS257, Package_SO:SOP-16_4.4x10.4mm_P1.27mm
- removed U18, U25, U27: 74LS245, Package_SO:TSSOP-20_4.4x5mm_P0.5mm
- added D45: LED, LED_SMD:LED_0805_2012Metric_Pad1.15x1.40mm_HandSolder, F.Cu at (48.3, 115.7)
- added D46: LED, LED_SMD:LED_0805_2012Metric_Pad1.15x1.40mm_HandSolder, F.Cu at (48.3, 118.8)
- added D47: LED, LED_SMD:LED_0805_2012Metric_Pad1.15x1.40mm_HandSolder, F.Cu at (48.3, 121.8)
- added D48: LED, LED_SMD:LED_0805_2012Metric_Pad1.15x1.40mm_HandSolder, F.Cu at (48.3, 124.8)
- added D49: LED, LED_SMD:LED_0603_1608Metric_Pad1.05x0.95mm_HandSolder, F.Cu at (48.1, 127.7)
- added R72: 560, Resistor_SMD:R_0603_1608Metric_Pad0.98x0.95mm_HandSolder, F.Cu at (29.4, 118.0)
- added R73: 560, Resistor_SMD:R_0603_1608Metric_Pad0.98x0.95mm_HandSolder, F.Cu at (29.4, 120.5)
- added R74: 10k, Resistor_SMD:R_0603_1608Metric_Pad0.98x0.95mm_HandSolder, F.Cu at (29.4, 123.0)
- added R75: 560, Resistor_SMD:R_0603_1608Metric_Pad0.98x0.95mm_HandSolder, F.Cu at (29.4, 125.5)
- added R76: 560, Resistor_SMD:R_0603_1608Metric_Pad0.98x0.95mm_HandSolder, F.Cu at (29.4, 128.0)
- added R77: 10k, Resistor_SMD:R_0603_1608Metric_Pad0.98x0.95mm_HandSolder, F.Cu at (29.4, 130.5)
- added R78: 560, Resistor_SMD:R_0603_1608Metric_Pad0.98x0.95mm_HandSolder, F.Cu at (29.4, 133.0)
- added SW22: SW_SPDT, Library:SW_K4625, F.Cu at (38.7, 128.5)
- added U28: 74LS06, Package_SO:SOIC-14_3.9x8.7mm_P1.27mm, F.Cu at (48.3, 98.7)
- added U29: 74LS06, Package_SO:SOIC-14_3.9x8.7mm_P1.27mm, F.Cu at (56.8, 98.7)
- added U30: 74LS06, Package_SO:SOIC-14_3.9x8.7mm_P1.27mm, F.Cu at (65.2, 98.7)
- added U31: 74LS06, Package_SO:SOIC-14_3.9x8.7mm_P1.27mm, F.Cu at (31.4, 109.1)
- added U32: 74LS06, Package_SO:SOIC-14_3.9x8.7mm_P1.27mm, F.Cu at (39.9, 109.1)
- added U33: 74LS06, Package_SO:SOIC-14_3.9x8.7mm_P1.27mm, F.Cu at (48.3, 109.1)
- moved U26 146.4 mm to (39.9, 98.7)
- moved U11 114.3 mm to (31.4, 98.7)
- moved SW13 60.3 mm to (38.7, 119.0)
- moved R12 29.8 mm to (29.4, 115.5)
Connections:
- D1 pad 1: D0IN -> Net-(D1-K)
- D2 pad 1: D1IN -> Net-(D2-K)
- D3 pad 1: D2IN -> Net-(D3-K)
- D4 pad 1: D3IN -> Net-(D4-K)
- D5 pad 1: D4IN -> Net-(D5-K)
- D6 pad 1: D5IN -> Net-(D6-K)
- D7 pad 1: D6IN -> Net-(D7-K)
- D8 pad 1: D7IN -> Net-(D8-K)
- J2 pad 44: VBUF -> SDA
- J2 pad 45: B2PHI2 -> SCL
- J2 pad 46: GND -> VBUF
- J2 pad 48: VCC -> B2PHI2
- R12 pad 1: /IO -> VCC
- R12 pad 2: GND -> /IO
- R41 pad 1: Net-(D18-K) -> Net-(D18-A)
- R41 pad 2: GND -> VCC
- R42 pad 1: Net-(D19-K) -> Net-(D19-A)
- R42 pad 2: GND -> VCC
- R43 pad 1: Net-(D20-K) -> Net-(D20-A)
- R43 pad 2: GND -> VCC
- R44 pad 1: Net-(D21-K) -> Net-(D21-A)
- R44 pad 2: GND -> VCC
- R45 pad 1: Net-(D22-K) -> Net-(D22-A)
- R45 pad 2: GND -> VCC
- R46 pad 1: Net-(D23-K) -> Net-(D23-A)
- R46 pad 2: GND -> VCC
- R47 pad 1: Net-(D24-K) -> Net-(D24-A)
- R47 pad 2: GND -> VCC
- R55 pad 1: Net-(D17-K) -> Net-(D17-A)
- R55 pad 2: GND -> VCC
- R56 pad 1: Net-(D29-K) -> Net-(D29-A)
- R56 pad 2: GND -> VCC
- R57 pad 1: Net-(D30-K) -> Net-(D30-A)
- R57 pad 2: GND -> VCC
- R58 pad 1: Net-(D31-K) -> Net-(D31-A)
- R58 pad 2: GND -> VCC
- R59 pad 1: Net-(D32-K) -> Net-(D32-A)
- R59 pad 2: GND -> VCC
- R60 pad 1: Net-(D33-K) -> Net-(D33-A)
- R60 pad 2: GND -> VCC
- R61 pad 1: Net-(D34-K) -> Net-(D34-A)
- R61 pad 2: GND -> VCC
- R62 pad 1: Net-(D35-K) -> Net-(D35-A)
- R62 pad 2: GND -> VCC
- R63 pad 1: Net-(D36-K) -> Net-(D36-A)
- R63 pad 2: GND -> VCC
- R64 pad 1: Net-(D37-K) -> Net-(D37-A)
- R64 pad 2: GND -> VCC
- R65 pad 1: Net-(D38-K) -> Net-(D38-A)
- R65 pad 2: GND -> VCC
- R66 pad 1: Net-(D39-K) -> Net-(D39-A)
- R66 pad 2: GND -> VCC
- R67 pad 1: Net-(D40-K) -> Net-(D40-A)
- R67 pad 2: GND -> VCC
- R68 pad 1: Net-(D41-K) -> Net-(D41-A)
- R68 pad 2: GND -> VCC
- R69 pad 1: Net-(D42-K) -> Net-(D42-A)
- R69 pad 2: GND -> VCC
- R70 pad 1: Net-(D43-K) -> Net-(D43-A)
- R70 pad 2: GND -> VCC
- R71 pad 1: Net-(D44-K) -> Net-(D44-A)
- R71 pad 2: GND -> VCC
- SW13 pad 1: VCC -> GND
- SW13 pad 2: /IO -> CLKIN
- U11 pad 1: Net-(U21A-~{Q}) -> unconnected-(U11-Pad1)
- U11 pad 10: /BUSEN -> (no net)
- U11 pad 11: Net-(U11-Pad11) -> (no net)
- U11 pad 12: Net-(U11-Pad12) -> (no net)
- U11 pad 13: Net-(D28-A) -> (no net)
- U11 pad 2: Net-(U22B-~{R}) -> unconnected-(U11-Pad2)
- U11 pad 3: Net-(U11-Pad3) -> unconnected-(U11-Pad3)
- U11 pad 4: Net-(U21B-~{Q}) -> unconnected-(U11-Pad4)
- U11 pad 6: Net-(U11-Pad6) -> unconnected-(U11-Pad6)
- U11 pad 8: /DOUTEN -> (no net)
- U11 pad 9: /WRITE -> (no net)
- U16 pad 9: unconnected-(U16-A7-Pad9) -> Net-(U16-A7)
- U17 pad 2: DOUT0 -> D0IN
- U17 pad 3: DOUT1 -> D1IN
- U17 pad 4: DOUT2 -> D2IN
- U17 pad 5: DOUT3 -> D3IN
- U17 pad 6: DOUT4 -> D4IN
- U17 pad 7: DOUT5 -> D5IN
- U17 pad 8: DOUT6 -> D6IN
- U17 pad 9: DOUT7 -> D7IN
- U19 pad 12: Net-(U11-Pad12) -> (no net)
- U19 pad 13: BRDY -> (no net)
- U19 pad 3: Net-(C4-Pad1) -> BPHI2
- U19 pad 4: CLKAL -> Net-(U22B-C)
- U19 pad 5: Net-(C5-Pad1) -> (no net)
- U19 pad 6: CLKAH -> (no net)
- U20 pad 1: Net-(U22B-Q) -> (no net)
- U20 pad 2: BPHI2 -> (no net)
- U20 pad 3: CLK_RD -> (no net)
- U20 pad 4: BPHI2 -> (no net)
- U20 pad 5: BPHI2 -> (no net)
- U20 pad 6: Net-(U22B-C) -> (no net)
- U21 pad 12: VCC -> Net-(U21A-Q)
- U21 pad 13: Net-(U21A-Q) -> /RES
- U22 pad 1: Net-(U21B-Q) -> /RES
- U22 pad 10: VCC -> unconnected-(U22B-~{S}-Pad10)
- U22 pad 12: Net-(U22B-D) -> unconnected-(U22B-D-Pad12)
- U22 pad 13: Net-(U22B-~{R}) -> Net-(U21A-C)
- U22 pad 2: VCC -> Net-(U21B-Q)
- U22 pad 8: /BUSEN -> unconnected-(U22B-~{Q}-Pad8)
- U22 pad 9: Net-(U22B-Q) -> unconnected-(U22B-Q-Pad9)
- U23 pad 1: Net-(U22B-~{R}) -> Net-(U23-Pad1)
- U23 pad 11: Net-(U11-Pad11) -> (no net)
- U23 pad 12: Net-(U22B-Q) -> (no net)
- U23 pad 13: Net-(U22B-D) -> (no net)
- U23 pad 5: CLKAL -> Net-(U21A-~{Q})
- U23 pad 6: Net-(U11-Pad3) -> Net-(U23-Pad1)
- U23 pad 8: CLKAH -> Net-(U21B-~{Q})
- U23 pad 9: Net-(U11-Pad6) -> Net-(U21B-Q)
- U26 pad 1: Net-(U22B-Q) -> (no net)
- U26 pad 10: unconnected-(U26-Pad10) -> Net-(R78-Pad1)
- U26 pad 11: Net-(R54-Pad2) -> Net-(U21B-~{Q})
- U26 pad 2: /BBE -> (no net)
- U26 pad 5: Net-(U21A-Q) -> Net-(U21A-~{Q})
- U26 pad 9: Net-(U21A-~{Q}) -> Net-(U21A-Q)
