File: Board/Board.kicad_sch (KiCad schematic)
At the start: 4 parts, among them J2 Conn_02x25_Odd_Even

Commit message: more work on the frontpanel
Parts:
- C1, C2: LCSC (none) -> C96123
- J2: LCSC (none) -> C30006
Connections:
- net /BBE: now also J2.10 (Pin_10)
- net /BIOSEL: now also J2.7 (Pin_7)
- net /BIRQ: now also J2.40 (Pin_40)
- net /BMEMSEL: now also J2.4 (Pin_4)
- net /BNMI: now also J2.37 (Pin_37)
- net /BRES: now also J2.43 (Pin_43)
- net B2PHI2: now also J2.45 (Pin_45)
- net B8PHI2: now also J2.47 (Pin_47)
- net BA0: now also J2.33 (Pin_33)
- net BA1: now also J2.29 (Pin_29)
- net BA10: now also J2.18 (Pin_18)
- net BA11: now also J2.14 (Pin_14)
- net BA12: now also J2.15 (Pin_15)
- net BA13: now also J2.11 (Pin_11)
- net BA14: now also J2.12 (Pin_12), J2.9 (Pin_9)
- net BA15: now also J2.8 (Pin_8)
- net BA17: now also J2.5 (Pin_5)
- net BA18: now also J2.6 (Pin_6)
- net BA19: now also J2.3 (Pin_3)
- net BA2: now also J2.30 (Pin_30)
- net BA3: now also J2.26 (Pin_26)
- net BA4: now also J2.27 (Pin_27)
- net BA5: now also J2.23 (Pin_23)
- net BA6: now also J2.24 (Pin_24)
- net BA7: now also J2.20 (Pin_20)
- net BA8: now also J2.21 (Pin_21)
- net BA9: now also J2.17 (Pin_17)
- net BD0: now also J2.34 (Pin_34)
- net BD1: now also J2.31 (Pin_31)
- net BD2: now also J2.28 (Pin_28)
- net BD3: now also J2.25 (Pin_25)
- net BD4: now also J2.22 (Pin_22)
- net BD5: now also J2.19 (Pin_19)
- net BD6: now also J2.16 (Pin_16)
- net BD7: now also J2.13 (Pin_13)
- net BPHI1: now also J2.39 (Pin_39)
- net BPHI2: now also J2.36 (Pin_36), J2.42 (Pin_42)
- net BR/-W: now also J2.35 (Pin_35)
- net BRDY: now also J2.38 (Pin_38)
- net BSYNC: now also J2.32 (Pin_32)
- net BV33: now also J2.41 (Pin_41)
- net GND: now also J2.46 (Pin_46), J2.49 (Pin_49)
- net VBUF: now also J2.44 (Pin_44)
- net VCC: now also J2.48 (Pin_48), J2.50 (Pin_50)
Other:
- note added: "CSA-FRONTPANEL-1.0A"
- note removed: "CBM-ULTIPET-V1.3A"

Commit message: More work
Connections:
- net B2PHI2: now also J2.48 (Pin_48); no longer J2.45 (Pin_45)
- net GND: no longer J2.46 (Pin_46)
- net VBUF: now also J2.46 (Pin_46); no longer J2.44 (Pin_44)
- net VCC: no longer J2.48 (Pin_48)
- new net SCL: J2.45 (Pin_45)
- new net SDA: J2.44 (Pin_44)
Changed lines of the file:
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@@
 	)
 	(junction
-		(at 264.16 128.905)
-		(diameter 0)
-		(color 0 0 0 0)
-	)
-	(junction
 		(at 147.32 78.74)
 		(diameter 0)
@@
 	)
 	(junction
-		(at 246.38 123.825)
-		(diameter 0)
-		(color 0 0 0 0)
-	)
-	(junction
 		(at 151.13 78.74)
 		(diameter 0)
@@
 	(wire
 		(pts
-			(xy 246.38 126.365) (xy 246.38 123.825)
+			(xy 242.57 118.745) (xy 251.46 118.745)
 		)
 		(stroke
@@
 	(wire
 		(pts
-			(xy 242.57 123.825) (xy 246.38 123.825)
-		)
-		(stroke
-			(width 0)
-			(type default)
-		)
-	)
-	(wire
-		(pts
 			(xy 147.32 78.74) (xy 151.13 78.74)
 		)
@@
 	(wire
 		(pts
-			(xy 217.805 116.205) (xy 229.87 116.205)
-		)
-		(stroke
-			(width 0)
-			(type default)
-		)
-	)
-	(wire
-		(pts
 			(xy 73.66 124.46) (xy 86.36 124.46)
 		)
@@
 	(wire
 		(pts
-			(xy 217.805 121.285) (xy 229.87 121.285)
-		)
-		(stroke
-			(width 0)
-			(type default)
-		)
-	)
-	(wire
-		(pts
 			(xy 151.13 55.88) (xy 157.48 55.88)
 		)
@@
 	(wire
 		(pts
-			(xy 246.38 123.825) (xy 252.73 123.825)
-		)
-		(stroke
-			(width 0)
-			(type default)
-		)
-	)
-	(wire
-		(pts
 			(xy 218.44 65.405) (xy 229.87 65.405)
 		)
@@
 	(wire
 		(pts
-			(xy 222.25 126.365) (xy 222.25 128.905)
+			(xy 222.25 126.365) (xy 222.25 127.635)
 		)
 		(stroke
@@
 	(wire
 		(pts
-			(xy 264.16 121.285) (xy 242.57 121.285)
-		)
-		(stroke
-			(width 0)
-			(type default)
-		)
-	)
-	(wire
-		(pts
 			(xy 86.36 60.96) (xy 73.66 60.96)
 		)
@@
 	(wire
 		(pts
-			(xy 264.16 121.285) (xy 264.16 131.445)
-		)
-		(stroke
-			(width 0)
-			(type default)
-		)
-	)
-	(wire
-		(pts
 			(xy 217.805 80.645) (xy 229.87 80.645)
 		)
@@
 	(wire
 		(pts
-			(xy 242.57 126.365) (xy 246.38 126.365)
+			(xy 242.57 126.365) (xy 251.46 126.365)
 		)
 		(stroke
@@
 	(wire
 		(pts
+			(xy 217.805 116.205) (xy 229.87 116.205)
+		)
+		(stroke
+			(width 0)
+			(type default)
+		)
+	)
+	(wire
+		(pts
 			(xy 86.36 116.84) (xy 73.66 116.84)
 		)
@@
 	(wire
 		(pts
-			(xy 217.805 67.945) (xy 229.87 67.945)
+			(xy 217.805 121.285) (xy 229.87 121.285)
 		)
 		(stroke
@@
 	(wire
 		(pts
-			(xy 86.36 111.76) (xy 73.66 111.76)
+			(xy 242.57 123.825) (xy 251.46 123.825)
 		)
 		(stroke
-			(width 0.1524)
-			(type solid)
+			(width 0)
+			(type default)
 		)
 	)
 	(wire
 		(pts
-			(xy 129.54 81.28) (xy 129.54 78.74)
+			(xy 217.805 67.945) (xy 229.87 67.945)
+		)
+		(stroke
+			(width 0)
+			(type default)
+		)
+	)
+	(wire
+		(pts
+			(xy 86.36 111.76) (xy 73.66 111.76)
 		)
 		(stroke
@@
 	(wire
 		(pts
-			(xy 254 65.405) (xy 254 64.77)
+			(xy 129.54 81.28) (xy 129.54 78.74)
 		)
 		(stroke
-			(width 0)
-			(type default)
+			(width 0.1524)
+			(type solid)
 		)
 	)
 	(wire
 		(pts
-			(xy 222.25 128.905) (xy 264.16 128.905)
+			(xy 254 65.405) (xy 254 64.77)
 		)
 		(stroke
@@
 	(wire
 		(pts
-			(xy 242.57 118.745) (xy 250.825 118.745)
+			(xy 217.805 118.745) (xy 229.87 118.745)
 		)
 		(stroke
@@
 	(wire
 		(pts
-			(xy 217.805 118.745) (xy 229.87 118.745)
+			(xy 242.57 121.285) (xy 251.46 121.285)
 		)
 		(stroke
@@
 	(global_label "VCC"
 		(shape bidirectional)
-		(at 252.73 123.825 0)
+		(at 251.46 126.365 0)
 		(fields_autoplaced yes)
 		(effects
@@
 		)
 		(property "Intersheetrefs" "${INTERSHEET_REFS}"
-			(at 260.3002 123.825 0)
+			(at 259.0302 126.365 0)
 			(hide yes)
 			(show_name no)
@@
 	(global_label "B2PHI2"
 		(shape bidirectional)
-		(at 217.805 121.285 180)
+		(at 251.46 123.825 0)
 		(fields_autoplaced yes)
 		(effects
@@
 				(size 1.2446 1.2446)
 			)
-			(justify right)
+			(justify left)
 		)
 		(property "Intersheetrefs" "${INTERSHEET_REFS}"
-			(at 207.0344 121.285 0)
+			(at 262.2306 123.825 0)
 			(hide yes)
 			(show_name no)
@@
 					(size 1.27 1.27)
 				)
-				(justify right)
+				(justify left)
 			)
 		)
@@
 		)
 	)
+	(global_label "SCL"
+		(shape bidirectional)
+		(at 217.805 121.285 180)
+		(fields_autoplaced yes)
+		(effects
+			(font
+				(size 1.2446 1.2446)
+			)
+			(justify right)
+		)
+		(property "Intersheetrefs" "${INTERSHEET_REFS}"
+			(at 210.3534 121.285 0)
+			(hide yes)
+			(show_name no)
+			(do_not_autoplace no)
+			(effects
+				(font
+					(size 1.27 1.27)
+				)
+				(justify right)
+			)
+		)
+	)
 	(global_label "BA1"
 		(shape bidirectional)
@@
 		)
 	)
+	(global_label "SDA"
+		(shape bidirectional)
+		(at 251.46 118.745 0)
+		(fields_autoplaced yes)
+		(effects
+			(font
+				(size 1.2446 1.2446)
+			)
+			(justify left)
+		)
+		(property "Intersheetrefs" "${INTERSHEET_REFS}"
+			(at 258.9709 118.745 0)
+			(hide yes)
+			(show_name no)
+			(do_not_autoplace no)
+			(effects
+				(font
+					(size 1.27 1.27)
+				)
+				(justify left)
+			)
+		)
+	)
 	(global_label "/BNMI"
 		(shape bidirectional)
@@
 	(global_label "VBUF"
 		(shape bidirectional)
-		(at 250.825 118.745 0)
+		(at 251.46 121.285 0)
 		(fields_autoplaced yes)
 		(effects
@@
 		)
 		(property "Intersheetrefs" "${INTERSHEET_REFS}"
-			(at 259.6992 118.745 0)
+			(at 260.3342 121.285 0)
 			(hide yes)
 			(show_name no)
@@
 	(symbol
 		(lib_id "cbm_ultipet_v1-eagle-import:GND")
-		(at 264.16 133.985 0)
+		(at 222.25 130.175 0)
 		(unit 1)
 		(body_style 1)
@@
 		(dnp no)
 		(property "Reference" "#GND061"
-			(at 264.16 133.985 0)
+			(at 222.25 130.175 0)
 			(hide yes)
 			(show_name no)
@@
 		)
 		(property "Value" "GND"
-			(at 261.62 136.525 0)
+			(at 219.71 132.715 0)
 			(show_name no)
 			(do_not_autoplace no)
@@
 		)
 		(property "Footprint" ""
-			(at 264.16 133.985 0)
+			(at 222.25 130.175 0)
 			(hide yes)
 			(show_name no)
@@
 		)
 		(property "Datasheet" ""
-			(at 264.16 133.985 0)
+			(at 222.25 130.175 0)
 			(hide yes)
 			(show_name no)
@@
 		)
 		(property "Description" ""
-			(at 264.16 133.985 0)
+			(at 222.25 130.175 0)
 			(hide yes)
 			(show_name no)
