File: Board/addrleds.kicad_sch (KiCad schematic)
At the start: 34 parts, among them U25 74LS245, U27 74LS245

Commit message: More work
Parts:
- removed U25, U27: 74LS245, Package_SO:TSSOP-20_4.4x5mm_P0.5mm, symbol 74xx:74LS245
- added U31, U32, U33: 74LS06, Package_SO:SOIC-14_3.9x8.7mm_P1.27mm, symbol 74xx:74LS06
Connections:
- net A0: now also U31.5
- net A1: now also U31.9
- net A10: now also U33.1
- net A11: now also U33.3
- net A12: now also U33.5
- net A13: now also U33.9
- net A14: now also U33.11
- net A15: now also U33.13
- net A2: now also U31.11
- net A3: now also U31.13
- net A4: now also U32.1
- net A5: now also U32.3
- net A6: now also U32.5
- net A7: now also U32.9
- net A8: now also U32.11
- net A9: now also U32.13
- net GND: now also U32.7 (GND), U33.7 (GND); no longer R56.2, R57.2, R58.2, R59.2, R60.2, R61.2, R62.2, R63.2, R64.2, R65.2, R66.2, R67.2, R68.2, R69.2, R70.2, R71.2
- net VCC: now also R56.2, R57.2, R58.2, R59.2, R60.2, R61.2, R62.2, R63.2, R64.2, R65.2, R66.2, R67.2, R68.2, R69.2, R70.2, R71.2, U32.14 (VCC), U33.14 (VCC)
- net at R57.1: now also D30.2 (A); no longer D30.1 (K)
- net at D29.2 (A): now also R56.1
- net at D31.2 (A): now also R58.1
- net at D32.2 (A): now also R59.1
- net at D33.2 (A): now also R60.1
- net at D34.2 (A): now also R61.1
- net at D35.2 (A): now also R62.1
- net at D36.2 (A): now also R63.1
- net at R64.1: now also D37.2 (A); no longer D37.1 (K)
- net at D41.1 (K): now also U31.12; no longer R68.1
- net at D41.2 (A): now also R68.1
- net at R65.1: now also D38.2 (A); no longer D38.1 (K)
- net at R71.1: now also D44.2 (A); no longer D44.1 (K)
- net at D36.1 (K): now also U32.10; no longer R63.1
- net at D40.1 (K): now also U32.2; no longer R67.1
- net at D39.2 (A): now also R66.1
- net at D40.2 (A): now also R67.1
- net at D42.2 (A): now also R69.1
- net at D43.2 (A): now also R70.1
- net at D33.1 (K): now also U33.4; no longer R60.1
- net at D35.1 (K): now also U32.12; no longer R62.1
- net at D34.1 (K): now also U33.2; no longer R61.1
- net at D39.1 (K): now also U32.4; no longer R66.1
- net at D29.1 (K): now also U33.12; no longer R56.1
- net at D42.1 (K): now also U31.10; no longer R69.1
- net at D43.1 (K): now also U31.8; no longer R70.1
- net at D31.1 (K): now also U33.8; no longer R58.1
- net at D32.1 (K): now also U33.6; no longer R59.1
- new net: D37.1 (K), U32.8
- new net: D38.1 (K), U32.6
- new net: D44.1 (K), U31.6
- new net: D30.1 (K), U33.10
Other:
- note added: "16/6 74LS06"
- moved on the sheet: D29, D30, D31, D32, D33, D34, D35, D36, D37, D38, D39, D40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
