File: Board/control.kicad_sch (KiCad schematic)
At the start: 22 parts, among them SW1 SW_SPST, SW18 SW_SPST, SW19 SW_SPST, SW20 SW_SPST, U11 74LS32, U19 74LS14, U20 74HCT00, U21 74HCT74, U22 74HCT74, U23 74HCT02

Commit message: more work on the frontpanel
Parts:
- added D25, D26, D27: LED, LED_SMD:LED_0603_1608Metric_Pad1.05x0.95mm_HandSolder, symbol Device:LED
- added D28: LED, LED_SMD:LED_0805_2012Metric_Pad1.15x1.40mm_HandSolder, symbol Device:LED
- added R48, R51, R52, R53: 560, Resistor_SMD:R_0603_1608Metric_Pad0.98x0.95mm_HandSolder, symbol Device:R
- added R49, R50, R54: 10k, Resistor_SMD:R_0603_1608Metric_Pad0.98x0.95mm_HandSolder, symbol Device:R
- added SW21: SW_SPDT, Library:SW_K4625, symbol Switch:SW_SPDT
- added unit 4 of U19
- added unit 2 of U19
- added unit 3 of U19
- added unit 1 of U22
- added unit 2 of U22
- added unit 4 of U23
- added U26: 74LS06, Package_SO:SOIC-14_3.9x8.7mm_P1.27mm, symbol 74xx:74LS06
- U11: footprint Package_CSP:Xilinx_CSG48_7.0x7.0mm_Layout7x7_P0.8mm -> Package_SO:SOIC-14_3.9x8.7mm_P1.27mm; LCSC (none) -> C5985
- U20: footprint Package_CSP:Xilinx_CSG48_7.0x7.0mm_Layout7x7_P0.8mm -> Package_SO:SOIC-14_3.9x8.7mm_P1.27mm; LCSC (none) -> C6764
- U21, U22: footprint Package_CSP:Xilinx_CSG48_7.0x7.0mm_Layout7x7_P0.8mm -> Package_SO:SOIC-14_3.9x8.7mm_P1.27mm; LCSC (none) -> C352961
- U23: footprint Package_CSP:Xilinx_CSG48_7.0x7.0mm_Layout7x7_P0.8mm -> Package_SO:SOIC-14_3.9x8.7mm_P1.27mm; LCSC (none) -> C471050
Connections:
- net /BBE: now also U26.2
- net BPHI2: now also U20.2, U20.4, U20.5; no longer U22.11 (C)
- net CLKAH: now also U19.6; no longer U19.6
- net CLKAL: now also U19.4; no longer U19.4
- net CLKD: now also U19.11, U19.8, U22.3 (C); no longer U19.13, U19.8
- net CLK_RD: now also U20.3
- net GND: now also U11.7 (GND), U21.7 (GND), U22.7 (GND), U23.7 (GND), R50.2, R53.2, U26.7 (GND)
- net RES: now also U26.3; no longer U19.11
- net SEL: now also U22.5 (Q); no longer U22.5 (Q)
- net VCC: now also U11.14 (VCC), U21.14 (VCC), U22.14 (VCC), U23.14 (VCC), D25.2 (A), D26.2 (A), D27.2 (A), R49.1, R54.1, SW21.1 (A), U22.10 (~{S}), U22.2 (D), U22.4 (~{S}), U26.14 (VCC); no longer U22.2 (D), U22.4 (~{S})
- net /BUSEN: now also U11.10, U22.8 (~{Q})
- net /DOUTEN: now also U11.8
- net /RES: now also R49.2, U26.4; no longer U19.10
- net CLKIN: now reaches R39.1, SW20.2 (B)
- net at C6.1, R39.2, R40.2: now also U19.9; no longer U19.9
- net at U21.11 (C), U21.3 (C): now also U19.10, U23.3; no longer U19.12, U23.3
- net at U21.13 (~{R}), U21.5 (Q): now also U26.5
- net at U11.4, U21.8 (~{Q}): now also U23.2; no longer U23.2
- net at U21.9 (Q): now also U22.1 (~{R}), U26.13; no longer U22.1 (~{R})
- net at C4.1, R35.2, R36.2: now also U19.3; no longer U19.3
- net at C5.1, R37.2, R38.2: now also U19.5; no longer U19.5
- net /RESIN: now reaches R33.1, SW1.2 (B)
- net at U11.11: now also U23.11
- net at U11.12: now also U19.12
- net at U11.13: now also D28.2 (A), R50.1, SW21.2 (B)
- net at U11.1, U21.6 (~{Q}): now also U26.9
- net /WRITE: now reaches U11.9
- new net: R52.1, U26.6
- new net: R54.2, U20.10, U20.12, U20.13, U20.9, U26.11
- new net: U11.2, U22.13 (~{R}), U23.1
- new net: U20.1, U22.9 (Q), U23.12, U26.1
- new net: U22.12 (D), U23.13
- new net: D28.1 (K), R53.1
- new net: R51.1, U26.8
- new net: D25.1 (K), R51.2
- new net: D26.1 (K), R52.2
- new net: U20.6, U22.11 (C)
- new net: D27.1 (K), R48.2
- new net: R48.1, U26.12
- new net BRDY: U19.13
- now unconnected: U11.5
Other:
- note added: "CSA-FRONTPANEL-1.0A"
- note added: "Phase D"
- note added: "Phase H"
- note added: "Phase L"
- note added: "Reset outside data clk then captures one bus cycle for transfer"
- moved on the sheet: C3, C4, C5, C6, R33, R34, R35, R36, R37, R38, R39, R40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

Commit message: More work
Parts:
- removed C4, C5: 100n, Capacitor_SMD:C_0603_1608Metric_Pad1.08x0.95mm_HandSolder, symbol Device:C
- removed D28: LED, LED_SMD:LED_0805_2012Metric_Pad1.15x1.40mm_HandSolder, symbol Device:LED
- removed R35, R37: 1k, Resistor_SMD:R_0603_1608Metric_Pad0.98x0.95mm_HandSolder, symbol Device:R
- removed R36, R38, R50: 10k, Resistor_SMD:R_0603_1608Metric_Pad0.98x0.95mm_HandSolder, symbol Device:R
- removed R53: 560, Resistor_SMD:R_0603_1608Metric_Pad0.98x0.95mm_HandSolder, symbol Device:R
- removed SW18, SW19: SW_SPST, Button_Switch_THT:SW_TH_Tactile_Omron_B3F-107x, symbol Switch:SW_SPST
- removed SW21: SW_SPDT, Library:SW_K4625, symbol Switch:SW_SPDT
- removed unit 4 of U11
- removed unit 1 of U11
- removed unit 2 of U11
- removed unit 3 of U11
- removed unit 3 of U19
- removed U20: 74HCT00, Package_SO:SOIC-14_3.9x8.7mm_P1.27mm, symbol 74xx:74HCT00
- removed unit 2 of U22
- removed unit 1 of U26
- added D49: LED, LED_SMD:LED_0603_1608Metric_Pad1.05x0.95mm_HandSolder, symbol Device:LED
- added R78: 560, Resistor_SMD:R_0603_1608Metric_Pad0.98x0.95mm_HandSolder, symbol Device:R
- added SW13: SW_SPDT, Library:SW_K4625, symbol Switch:SW_SPDT
- added U20: 74HCT00, Package_SO:SOIC-14_3.9x8.7mm_P1.27mm, symbol 74xx:74HCT00
Connections:
- net CLKAH is gone; now on an unnamed net: U23.8
- net CLKD: now also U19.11; no longer U19.11
- net CLKIN: now also SW13.2 (B)
- net GND: now also SW13.1 (A), U20.7 (GND)
- net VCC: now also D49.2 (A), U20.14 (VCC); no longer U21.12 (D), U22.2 (D)
- net /RES: now also U21.13 (~{R}), U22.1 (~{R})
- net CLK: now reaches U21.11 (C), U21.3 (C), U23.3
- net CLK: now also U19.10; no longer U19.10
- net at U21.8 (~{Q}), U23.2: now also U26.11
- net at U21.9 (Q), U26.13: now also U22.2 (D), U23.9; no longer U22.1 (~{R})
- net at R54.2: now also U20.12, U20.13; no longer U26.11
- net /DCLK: now reaches U23.6
- net /DCLK: now also U23.1
- net at U21.6 (~{Q}): now also U23.5, U26.5; no longer U26.9
- net at U26.10: now also R78.1
- removed net BRDY: U19.13
- removed net CLKAL: U19.4, U23.5
- new net: U21.12 (D), U21.5 (Q), U26.9
- new net: D49.1 (K), R78.2
Other:
- note added: "AH Green"
- note added: "AH Red"
- note added: "AL Green"
- note added: "AL Red"
- note removed: "Phase D"
- note removed: "Phase H"
- note removed: "Phase L"
- note removed: "Reset outside data clk then captures one bus cycle for transfer"
- moved on the sheet: C3, C6, D25, D26, D27, R33, R34, R39, R40, R48, R49, R51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
