File: Board/data.kicad_sch (KiCad schematic)
At the start: 5 parts, among them U14 74LS245, U15 74LS245, U16 74LS245, U17 74LS245, U24 74LS273

Commit message: more work on the frontpanel
Other:
- note added: "CSA-FRONTPANEL-1.0A"
Changed lines of the file:
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@@
 	(generator_version "10.0")
 	(paper "A4")
+	(text "CSA-FRONTPANEL-1.0A"
+		(exclude_from_sim no)
+		(at 192.405 177.165 0)
+		(effects
+			(font
+				(size 3.81 3.2385)
+			)
+			(justify left bottom)
+		)
+	)
 	(junction
 		(at 214.63 48.895)

Commit message: More work
Parts:
- added R77: 10k, Resistor_SMD:R_0603_1608Metric_Pad0.98x0.95mm_HandSolder, symbol Device:R
- added U27: 74LS273, Package_SO:TSSOP-20_4.4x6.5mm_P0.65mm, symbol 74xx:74LS273
Connections:
- net CLK_RD: now also U27.11 (Cp); no longer U24.11 (Cp)
- net DIN0: now also U27.2 (Q0); no longer U24.2 (Q0)
- net DIN1: now also U27.5 (Q1); no longer U24.5 (Q1)
- net DIN2: now also U27.6 (Q2); no longer U24.6 (Q2)
- net DIN3: now also U27.9 (Q3); no longer U24.9 (Q3)
- net DIN4: now also U27.12 (Q4); no longer U24.12 (Q4)
- net DIN5: now also U27.15 (Q5); no longer U24.15 (Q5)
- net DIN6: now also U27.16 (Q6); no longer U24.16 (Q6)
- net DIN7: now also U27.19 (Q7); no longer U24.19 (Q7)
- net GND: now also R77.2, U27.10 (GND)
- net VCC: now also U27.20 (VCC)
- net /RES: now also U27.1 (~{Mr})
- net at U16.9 (A7): now also R77.1
- new net: U24.12 (Q4), U27.13 (D4)
- new net: U24.15 (Q5), U27.14 (D5)
- new net: U24.16 (Q6), U27.17 (D6)
- new net: U24.19 (Q7), U27.18 (D7)
- new net: U24.2 (Q0), U27.3 (D0)
- new net: U24.5 (Q1), U27.4 (D1)
- new net: U24.6 (Q2), U27.7 (D2)
- new net: U24.9 (Q3), U27.8 (D3)
- new net /PHI2: U24.11 (Cp)
Other:
- moved on the sheet: U17, U24
