File: Board/panel.kicad_sch (KiCad schematic)
At the start: 0 parts

Commit message: More work
Other:
- note added: "4 LED A23-16"
- note added: "4 Toggle for A16-23"
- note added: "Toggle for control. and Control LEDS"
- note removed: "8 Toggle for control. A16-23"
- note removed: "8 control input monitor LEDs"
Changed lines of the file:
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@@
 	(paper "A4")
 	(circle
-		(center 124.46 86.995)
+		(center 146.05 86.995)
 		(radius 1.7961)
 		(stroke
@@
 	)
 	(rectangle
-		(start 151.13 116.84)
-		(end 156.845 121.285)
-		(stroke
-			(width 0)
-			(type default)
-		)
-		(fill
-			(type none)
-		)
-	)
-	(rectangle
-		(start 61.595 93.345)
-		(end 117.475 97.79)
-		(stroke
-			(width 0)
-			(type default)
-		)
-		(fill
-			(type none)
-		)
-	)
-	(rectangle
-		(start 151.765 123.825)
-		(end 157.48 133.985)
-		(stroke
-			(width 0)
-			(type default)
-		)
-		(fill
-			(type none)
-		)
-	)
-	(rectangle
-		(start 89.535 123.825)
-		(end 145.415 133.985)
+		(start 245.745 99.695)
+		(end 251.46 104.14)
+		(stroke
+			(width 0)
+			(type default)
+		)
+		(fill
+			(type none)
+		)
+	)
+	(rectangle
+		(start 149.225 99.695)
+		(end 205.105 104.14)
+		(stroke
+			(width 0)
+			(type default)
+		)
+		(fill
+			(type none)
+		)
+	)
+	(rectangle
+		(start 246.38 106.68)
+		(end 252.095 116.84)
+		(stroke
+			(width 0)
+			(type default)
+		)
+		(fill
+			(type none)
+		)
+	)
+	(rectangle
+		(start 52.705 109.22)
+		(end 205.74 120.015)
 		(stroke
 			(width 0)
@@
 	)
 	(rectangle
-		(start 127.635 84.455)
-		(end 183.515 88.9)
-		(stroke
-			(width 0)
-			(type default)
-		)
-		(fill
-			(type none)
-		)
-	)
-	(rectangle
-		(start 89.535 116.84)
-		(end 145.415 121.285)
-		(stroke
-			(width 0)
-			(type default)
-		)
-		(fill
-			(type none)
-		)
-	)
-	(rectangle
-		(start 131.445 102.87)
-		(end 137.16 107.315)
-		(stroke
-			(width 0)
-			(type default)
-		)
-		(fill
-			(type none)
-		)
-	)
-	(rectangle
-		(start 61.595 100.33)
-		(end 117.475 110.49)
+		(start 149.225 84.455)
+		(end 205.105 88.9)
+		(stroke
+			(width 0)
+			(type default)
+		)
+		(fill
+			(type none)
+		)
+	)
+	(rectangle
+		(start 52.07 93.345)
+		(end 73.66 103.505)
 		(stroke
 			(width 0)
@@
 	)
 	(rectangle
-		(start 142.24 102.87)
-		(end 147.955 107.315)
-		(stroke
-			(width 0)
-			(type default)
-		)
-		(fill
-			(type none)
-		)
-	)
-	(rectangle
-		(start 127.635 93.345)
-		(end 183.515 97.79)
+		(start 226.06 85.725)
+		(end 231.775 90.17)
+		(stroke
+			(width 0)
+			(type default)
+		)
+		(fill
+			(type none)
+		)
+	)
+	(rectangle
+		(start 83.185 93.345)
+		(end 139.065 103.505)
+		(stroke
+			(width 0)
+			(type solid)
+		)
+		(fill
+			(type none)
+		)
+	)
+	(rectangle
+		(start 236.855 85.725)
+		(end 242.57 90.17)
+		(stroke
+			(width 0)
+			(type default)
+		)
+		(fill
+			(type none)
+		)
+	)
+	(rectangle
+		(start 149.225 92.075)
+		(end 205.105 96.52)
 		(stroke
 			(width 0)
@@
 	)
 	(circle
-		(center 57.785 86.995)
+		(center 79.375 86.995)
 		(radius 1.7961)
 		(stroke
@@
 	)
 	(rectangle
-		(start 160.02 116.84)
-		(end 165.735 121.285)
-		(stroke
-			(width 0)
-			(type default)
-		)
-		(fill
-			(type none)
-		)
-	)
-	(rectangle
-		(start 61.595 84.455)
-		(end 117.475 88.9)
+		(start 254.635 99.695)
+		(end 260.35 104.14)
+		(stroke
+			(width 0)
+			(type default)
+		)
+		(fill
+			(type none)
+		)
+	)
+	(rectangle
+		(start 83.185 84.455)
+		(end 139.065 88.9)
+		(stroke
+			(width 0)
+			(type default)
+		)
+		(fill
+			(type none)
+		)
+	)
+	(rectangle
+		(start 52.07 84.455)
+		(end 73.66 88.9)
 		(stroke
 			(width 0)
@@
 	)
 	(circle
-		(center 124.46 95.25)
+		(center 146.05 93.98)
 		(radius 1.7961)
 		(stroke
@@
 	)
 	(rectangle
-		(start 160.02 124.46)
-		(end 165.735 128.905)
+		(start 254.635 107.315)
+		(end 260.35 111.76)
 		(stroke
 			(width 0)
@@
 	(text "CONT"
 		(exclude_from_sim no)
-		(at 154.305 128.27 0)
-		(effects
-			(font
-				(size 1.27 1.27)
-			)
-		)
-	)
-	(text "8 Toggle for control. A16-23"
-		(exclude_from_sim no)
-		(at 115.57 129.54 0)
+		(at 248.92 111.125 0)
+		(effects
+			(font
+				(size 1.27 1.27)
+			)
+		)
+	)
+	(text "Toggle for control. \nand Control LEDS"
+		(exclude_from_sim no)
+		(at 129.54 114.935 0)
 		(effects
 			(font
@@
 	(text "DCLK"
 		(exclude_from_sim no)
-		(at 145.415 105.41 0)
+		(at 240.03 88.265 0)
 		(effects
 			(font
@@
 	(text "8 LED A15-8"
 		(exclude_from_sim no)
-		(at 87.63 86.995 0)
+		(at 109.22 86.995 0)
 		(effects
 			(font
@@
 	(text "RES"
 		(exclude_from_sim no)
-		(at 134.62 105.41 0)
+		(at 229.235 88.265 0)
 		(effects
 			(font
@@
 	(text "L"
 		(exclude_from_sim no)
-		(at 57.785 86.995 0)
-		(effects
-			(font
-				(size 1.27 1.27)
-			)
-		)
-	)
-	(text "8 control input monitor LEDs"
-		(exclude_from_sim no)
-		(at 115.57 119.38 0)
+		(at 79.375 86.995 0)
+		(effects
+			(font
+				(size 1.27 1.27)
+			)
+		)
+	)
+	(text "4 LED A23-16"
+		(exclude_from_sim no)
+		(at 62.865 86.995 0)
 		(effects
 			(font
@@
 	(text "AL"
 		(exclude_from_sim no)
-		(at 163.195 119.38 0)
+		(at 257.81 102.235 0)
+		(effects
+			(font
+				(size 1.27 1.27)
+			)
+		)
+	)
+	(text "4 Toggle for A16-23"
+		(exclude_from_sim no)
+		(at 62.865 99.06 0)
 		(effects
 			(font
@@
 	(text "8 LED A7-0"
 		(exclude_from_sim no)
-		(at 153.67 86.995 0)
+		(at 175.26 86.995 0)
 		(effects
 			(font
@@
 	(text "AH"
 		(exclude_from_sim no)
-		(at 163.195 127 0)
+		(at 257.81 109.855 0)
 		(effects
 			(font
@@
 	(text "8 data input monitor LEDs"
 		(exclude_from_sim no)
-		(at 87.63 95.885 0)
+		(at 175.26 102.235 0)
 		(effects
 			(font
@@
 	(text "H"
 		(exclude_from_sim no)
-		(at 124.46 86.995 0)
+		(at 146.05 86.995 0)
 		(effects
 			(font
@@
 	(text "D"
 		(exclude_from_sim no)
-		(at 124.46 95.25 0)
+		(at 146.05 93.98 0)
 		(effects
 			(font
@@
 	(text "CONT\nLED"
 		(exclude_from_sim no)
-		(at 154.305 119.38 0)
+		(at 248.92 102.235 0)
 		(effects
 			(font
@@
 	(text "8 LED D7-0 IN"
 		(exclude_from_sim no)
-		(at 153.67 95.885 0)
+		(at 175.26 94.615 0)
 		(effects
 			(font
@@
 	(text "8 Toggle for Data input"
 		(exclude_from_sim no)
-		(at 87.63 106.045 0)
-		(effects
-			(font
+		(at 109.22 99.06 0)
+		(effects
+			(font
